File: bobbycar.kicad_pcb (KiCad board)
At the start: 2 copper layers, 61.9 x 26.9 mm, 29 parts, among them J1 Conn_01x04, J2 Conn_01x04, J3 Screw_Terminal_01x02, J4 Screw_Terminal_01x02, J5 Screw_Terminal_01x02, J6 Conn_01x04, U1 L7805

Commit message: UPDATED pcb files
Parts:
- C1, C2, C3, C4: footprint Capacitors_THT:C_Disc_D5.0mm_W2.5mm_P2.50mm -> Capacitors_THT:C_Disc_D5.0mm_W2.5mm_P5.00mm
- U1: value L7805 -> L7805SOT89
- moved J2 7.55 mm to (104.5, 102.0), turned to 270 degrees
- moved J1 7.55 mm to (104.5, 88.5), turned to 270 degrees
- moved C4 2.01 mm to (138.0, 88.8)
- moved C8 1.95 mm to (141.5, 101.0)
- moved C7 1.82 mm to (141.5, 95.9)
- moved C3 1.66 mm to (126.1, 96.1)
- moved C2 1.65 mm to (144.0, 101.0)
- moved C6 1.08 mm to (135.3, 98.6)
- moved C1 0.95 mm to (139.0, 95.9)
- moved C5 0.73 mm to (127.5, 99.6)
- moved U1 0.66 mm to (133.0, 91.8), turned to 0 degrees
- moved G*** 0.18 mm to (132.6, 106.2)
- moved J6 0.05 mm to (158.3, 98.8)
Connections:
- J1 pad 1: GND -> Net-(D1-Pad2)
- J1 pad 2: RX.1 -> TX.1
- J1 pad 3: TX.1 -> RX.1
- J1 pad 4: Net-(D1-Pad2) -> GND
- J2 pad 1: GND -> Net-(D2-Pad2)
- J2 pad 2: RX -> TX
- J2 pad 3: TX -> RX
- J2 pad 4: Net-(D2-Pad2) -> GND
- U1 pad 1: VDD -> VCC
- U1 pad 3: VCC -> VDD
Routing:
- net VCC: track 28.4 -> 32.2 mm
- net TX: track 94.8 -> 93.0 mm
- net Net-(D1-Pad2): track 8.05 -> 6.66 mm
- net RX: track 106.1 -> 104.9 mm
- net RX.1: track 13.1 -> 12.2 mm
- net Net-(D2-Pad2): track 8.36 -> 8.91 mm
- net TX.1: track 7.84 -> 7.29 mm
- net GND: vias 11 -> 14
Other:
- board size 61.9 x 26.9 mm -> 61.7 x 26.9 mm
- board text added: "ADC"
- board text added: "I²C"
