File: bobbycar.sch (KiCad schematic (older format))
At the start: 28 parts, among them J1 Conn_01x04, J2 Conn_01x04, J3 Screw_Terminal_01x02, J4 Screw_Terminal_01x02, J5 Screw_Terminal_01x02, J6 Conn_01x04, U1 L7805

Commit message: UPDATED pcb files
Parts:
- removed U1: L7805, TO_SOT_Packages_SMD:SOT-89-3_Handsoldering, symbol regul:L7805
- added U1: L7805SOT89, TO_SOT_Packages_SMD:SOT-89-3_Handsoldering, symbol regul_eigen:L7805SOT89
- C1, C2, C3, C4: footprint Capacitors_THT:C_Disc_D5.0mm_W2.5mm_P2.50mm -> Capacitors_THT:C_Disc_D5.0mm_W2.5mm_P5.00mm
Connections:
- wire segments 20 -> 24
Changed lines of the file:
@@
 F 0 "C4" H 5665 3646 50  0000 L CNN
 F 1 "1uF" H 5665 3555 50  0000 L CNN
-F 2 "Capacitors_THT:C_Disc_D5.0mm_W2.5mm_P2.50mm" H 5588 3450 50  0001 C CNN
+F 2 "Capacitors_THT:C_Disc_D5.0mm_W2.5mm_P5.00mm" H 5588 3450 50  0001 C CNN
 F 3 "" H 5550 3600 50  0001 C CNN
 	1    5550 3600
@@
 F 0 "C3" H 4865 3646 50  0000 L CNN
 F 1 "1uF" H 4865 3555 50  0000 L CNN
-F 2 "Capacitors_THT:C_Disc_D5.0mm_W2.5mm_P2.50mm" H 4788 3450 50  0001 C CNN
+F 2 "Capacitors_THT:C_Disc_D5.0mm_W2.5mm_P5.00mm" H 4788 3450 50  0001 C CNN
 F 3 "" H 4750 3600 50  0001 C CNN
 	1    4750 3600
@@
 L conn:Conn_01x04 J2
 U 1 1 5AB40975
-P 3150 3550
-F 0 "J2" H 3070 3125 50  0000 C CNN
-F 1 "Conn_01x04" H 3070 3216 50  0000 C CNN
-F 2 "Connectors_JST:JST_XH_B04B-XH-A_04x2.50mm_Straight" H 3150 3550 50  0001 C CNN
-F 3 "~" H 3150 3550 50  0001 C CNN
-	1    3150 3550
+P 2900 3550
+F 0 "J2" H 2820 3125 50  0000 C CNN
+F 1 "Conn_01x04" H 2820 3216 50  0000 C CNN
+F 2 "Connectors_JST:JST_XH_B04B-XH-A_04x2.50mm_Straight" H 2900 3550 50  0001 C CNN
+F 3 "~" H 2900 3550 50  0001 C CNN
+	1    2900 3550
 	-1   0    0    1
 $EndComp
@@
 L power:GND #PWR0102
 U 1 1 5AB40AE8
-P 3350 3650
-F 0 "#PWR0102" H 3350 3400 50  0001 C CNN
-F 1 "GND" H 3355 3477 50  0000 C CNN
-F 2 "" H 3350 3650 50  0001 C CNN
-F 3 "" H 3350 3650 50  0001 C CNN
-	1    3350 3650
-	1    0    0    -1
+P 3100 3350
+F 0 "#PWR0102" H 3100 3100 50  0001 C CNN
+F 1 "GND" H 3105 3177 50  0000 C CNN
+F 2 "" H 3100 3350 50  0001 C CNN
+F 3 "" H 3100 3350 50  0001 C CNN
+	1    3100 3350
+	-1   0    0    1
 $EndComp
 $Comp
@@
 L power:VDD #PWR0108
 U 1 1 5AB40D07
-P 3350 3050
-F 0 "#PWR0108" H 3350 2900 50  0001 C CNN
-F 1 "VDD" H 3367 3223 50  0000 C CNN
-F 2 "" H 3350 3050 50  0001 C CNN
-F 3 "" H 3350 3050 50  0001 C CNN
-	1    3350 3050
-	1    0    0    -1
+P 3100 3950
+F 0 "#PWR0108" H 3100 3800 50  0001 C CNN
+F 1 "VDD" H 3117 4123 50  0000 C CNN
+F 2 "" H 3100 3950 50  0001 C CNN
+F 3 "" H 3100 3950 50  0001 C CNN
+	1    3100 3950
+	-1   0    0    1
 $EndComp
 Wire Wire Line
 	4700 3450 4750 3450
-Wire Wire Line
-	4850 3450 4750 3450
-Connection ~ 4750 3450
 Wire Wire Line
 	5450 3450 5550 3450
@@
 F 0 "C2" H 3542 3696 50  0000 L CNN
 F 1 "C_Small" H 3542 3605 50  0000 L CNN
-F 2 "Capacitors_THT:C_Disc_D5.0mm_W2.5mm_P2.50mm" H 3450 3650 50  0001 C CNN
+F 2 "Capacitors_THT:C_Disc_D5.0mm_W2.5mm_P5.00mm" H 3450 3650 50  0001 C CNN
 F 3 "" H 3450 3650 50  0001 C CNN
 	1    3450 3650
@@
 F 0 "C1" H 3542 3396 50  0000 L CNN
 F 1 "C_Small" H 3542 3305 50  0000 L CNN
-F 2 "Capacitors_THT:C_Disc_D5.0mm_W2.5mm_P2.50mm" H 3450 3350 50  0001 C CNN
+F 2 "Capacitors_THT:C_Disc_D5.0mm_W2.5mm_P5.00mm" H 3450 3350 50  0001 C CNN
 F 3 "" H 3450 3350 50  0001 C CNN
 	1    3450 3350
@@
 $EndComp
 Wire Wire Line
-	3350 3450 3450 3450
-Wire Wire Line
 	3600 3450 3450 3450
-Connection ~ 3450 3450
-Wire Wire Line
-	3350 3550 3450 3550
 Wire Wire Line
 	3600 3550 3450 3550
-Connection ~ 3450 3550
 Text GLabel 4100 3450 2    50   Input ~ 0
 TX
@@
 L device:D D2
 U 1 1 5AB41CA8
-P 3350 3200
-F 0 "D2" V 3304 3279 50  0000 L CNN
-F 1 "D" V 3395 3279 50  0000 L CNN
-F 2 "Diodes_THT:D_DO-41_SOD81_P7.62mm_Horizontal" H 3350 3200 50  0001 C CNN
-F 3 "" H 3350 3200 50  0001 C CNN
-	1    3350 3200
-	0    1    1    0
+P 3100 3800
+F 0 "D2" V 3054 3879 50  0000 L CNN
+F 1 "D" V 3145 3879 50  0000 L CNN
+F 2 "Diodes_THT:D_DO-41_SOD81_P7.62mm_Horizontal" H 3100 3800 50  0001 C CNN
+F 3 "" H 3100 3800 50  0001 C CNN
+	1    3100 3800
+	0    -1   -1   0
 $EndComp
 $Comp
@@
 L device:D D1
 U 1 1 5AB41BB2
-P 2800 3200
-F 0 "D1" V 2754 3279 50  0000 L CNN
-F 1 "D" V 2845 3279 50  0000 L CNN
-F 2 "Diodes_THT:D_DO-41_SOD81_P7.62mm_Horizontal" H 2800 3200 50  0001 C CNN
-F 3 "" H 2800 3200 50  0001 C CNN
-	1    2800 3200
-	0    1    1    0
-$EndComp
-Text GLabel 2800 3550 2    50   Input ~ 0
+P 2600 3800
+F 0 "D1" V 2554 3879 50  0000 L CNN
+F 1 "D" V 2645 3879 50  0000 L CNN
+F 2 "Diodes_THT:D_DO-41_SOD81_P7.62mm_Horizontal" H 2600 3800 50  0001 C CNN
+F 3 "" H 2600 3800 50  0001 C CNN
+	1    2600 3800
+	0    -1   -1   0
+$EndComp
+Text GLabel 2600 3450 2    50   Input ~ 0
 RX.1
-Text GLabel 2800 3450 2    50   Input ~ 0
+Text GLabel 2600 3550 2    50   Input ~ 0
 TX.1
 $Comp
 L power:VDD #PWR0109
 U 1 1 5AB40D38
-P 2800 3050
-F 0 "#PWR0109" H 2800 2900 50  0001 C CNN
-F 1 "VDD" H 2817 3223 50  0000 C CNN
-F 2 "" H 2800 3050 50  0001 C CNN
-F 3 "" H 2800 3050 50  0001 C CNN
-	1    2800 3050
-	1    0    0    -1
+P 2600 3950
+F 0 "#PWR0109" H 2600 3800 50  0001 C CNN
+F 1 "VDD" H 2617 4123 50  0000 C CNN
+F 2 "" H 2600 3950 50  0001 C CNN
+F 3 "" H 2600 3950 50  0001 C CNN
+	1    2600 3950
+	-1   0    0    1
 $EndComp
 $Comp
 L power:GND #PWR0101
 U 1 1 5AB40AB7
-P 2800 3650
-F 0 "#PWR0101" H 2800 3400 50  0001 C CNN
-F 1 "GND" H 2805 3477 50  0000 C CNN
-F 2 "" H 2800 3650 50  0001 C CNN
-F 3 "" H 2800 3650 50  0001 C CNN
-	1    2800 3650
-	1    0    0    -1
+P 2600 3350
+F 0 "#PWR0101" H 2600 3100 50  0001 C CNN
+F 1 "GND" H 2605 3177 50  0000 C CNN
+F 2 "" H 2600 3350 50  0001 C CNN
+F 3 "" H 2600 3350 50  0001 C CNN
+	1    2600 3350
+	-1   0    0    1
 $EndComp
 $Comp
 L conn:Conn_01x04 J1
 U 1 1 5AB40A05
-P 2600 3550
-F 0 "J1" H 2520 3125 50  0000 C CNN
-F 1 "Conn_01x04" H 2520 3216 50  0000 C CNN
-F 2 "Connectors_JST:JST_XH_B04B-XH-A_04x2.50mm_Straight" H 2600 3550 50  0001 C CNN
-F 3 "~" H 2600 3550 50  0001 C CNN
-	1    2600 3550
+P 2400 3550
+F 0 "J1" H 2320 3125 50  0000 C CNN
+F 1 "Conn_01x04" H 2320 3216 50  0000 C CNN
+F 2 "Connectors_JST:JST_XH_B04B-XH-A_04x2.50mm_Straight" H 2400 3550 50  0001 C CNN
+F 3 "~" H 2400 3550 50  0001 C CNN
+	1    2400 3550
 	-1   0    0    1
 $EndComp
@@
 	1    0    0    -1
 $EndComp
-$Comp
-L regul:L7805 U1
-U 1 1 5AD34B6F
-P 5150 3450
-F 0 "U1" H 5150 3692 50  0000 C CNN
-F 1 "L7805" H 5150 3601 50  0000 C CNN
-F 2 "TO_SOT_Packages_SMD:SOT-89-3_Handsoldering" H 5175 3300 50  0001 L CIN
-F 3 "http://www.st.com/content/ccc/resource/technical/document/datasheet/41/4f/b3/b0/12/d4/47/88/CD00000444.pdf/files/CD00000444.pdf/jcr:content/translations/en.CD00000444.pdf" H 5150 3400 50  0001 C CNN
-	1    5150 3450
-	1    0    0    -1
-$EndComp
 Wire Wire Line
 	4100 3450 3900 3450
@@
 Text GLabel 4800 5200 0    50   Input ~ 0
 RX
+Wire Wire Line
+	4850 3450 4750 3450
+Connection ~ 4750 3450
+$Comp
+L regul_eigen:L7805SOT89 U1
+U 1 1 5AE0F904
+P 5150 3450
+F 0 "U1" H 5150 3692 50  0000 C CNN
+F 1 "L7805SOT89" H 5150 3601 50  0000 C CNN
+F 2 "TO_SOT_Packages_SMD:SOT-89-3_Handsoldering" H 5175 3300 50  0001 L CIN
+F 3 "http://www.st.com/content/ccc/resource/technical/document/datasheet/41/4f/b3/b0/12/d4/47/88/CD00000444.pdf/files/CD00000444.pdf/jcr:content/translations/en.CD00000444.pdf" H 5150 3400 50  0001 C CNN
+	1    5150 3450
+	1    0    0    -1
+$EndComp
+Wire Wire Line
+	3450 3500 3450 3450
+Connection ~ 3450 3450
+Wire Wire Line
+	3450 3500 3100 3500
+Wire Wire Line
+	3100 3500 3100 3550
+Wire Wire Line
+	3450 3550 3200 3550
+Wire Wire Line
+	3200 3550 3200 3450
+Wire Wire Line
+	3200 3450 3100 3450
+Connection ~ 3450 3550
 $EndSCHEMATC

Commit message: fixed library names
Parts:
- C1, C2, C7, C8: symbol device:C_Small -> Device:C_Small
- C3, C4: symbol device:C -> Device:C
- C5, C6: symbol device:CP -> Device:CP
- D1, D2: symbol device:D -> Device:D
- D3: symbol device:LED -> Device:LED
- J1, J2, J6: symbol conn:Conn_01x04 -> Connector_Generic:Conn_01x04
- J3, J4, J5: symbol conn:Screw_Terminal_01x02 -> Connector:Screw_Terminal_01x02
- JP1, JP2: symbol device:Jumper_NC_Dual -> Device:Jumper_NC_Dual
- R1, R2, R6, R7: symbol device:R_Small -> Device:R_Small
- R3, R4, R5: symbol device:R -> Device:R
- U1: symbol regul_eigen:L7805SOT89 -> Regulator_Linear:L7805
- UART1: symbol conn:Conn_01x03 -> Connector_Generic:Conn_01x03
Connections:
- wire segments 24 -> 13
Changed lines of the file:
@@
 EESchema Schematic File Version 4
-LIBS:bobbycar-cache
 EELAYER 26 0
 EELAYER END
@@
 $EndDescr
 $Comp
-L device:C C4
+L Device:C C4
 U 1 1 5AB407B6
 P 5550 3600
@@
 $EndComp
 $Comp
-L device:C C3
+L Device:C C3
 U 1 1 5AB40828
 P 4750 3600
@@
 $EndComp
 $Comp
-L conn:Conn_01x04 J2
+L Connector_Generic:Conn_01x04 J2
 U 1 1 5AB40975
 P 2900 3550
@@
 	-1   0    0    1
 $EndComp
-Wire Wire Line
-	4700 3450 4750 3450
-Wire Wire Line
-	5450 3450 5550 3450
-Connection ~ 5550 3450
-Wire Wire Line
-	5550 3450 5600 3450
-$Comp
-L device:C_Small C2
+$Comp
+L Device:C_Small C2
 U 1 1 5AB411A2
 P 3450 3650
@@
 $EndComp
 $Comp
-L device:C_Small C1
+L Device:C_Small C1
 U 1 1 5AB411E3
 P 3450 3350
@@
 $EndComp
 $Comp
-L device:R_Small R2
+L Device:R_Small R2
 U 1 1 5AB412F6
 P 3600 3650
@@
 $EndComp
 $Comp
-L device:R_Small R1
+L Device:R_Small R1
 U 1 1 5AB41339
 P 3600 3350
@@
 	-1   0    0    1
 $EndComp
-Wire Wire Line
-	3600 3450 3450 3450
-Wire Wire Line
-	3600 3550 3450 3550
 Text GLabel 4100 3450 2    50   Input ~ 0
 TX
@@
 RX
 $Comp
-L device:D D2
+L Device:D D2
 U 1 1 5AB41CA8
 P 3100 3800
@@
 $EndComp
 $Comp
-L device:LED D3
+L Device:LED D3
 U 1 1 5AB41F7D
 P 4900 4450
@@
 $EndComp
 $Comp
-L device:R R3
+L Device:R R3
 U 1 1 5AB42057
 P 4600 4450
@@
 $EndComp
 $Comp
-L conn:Screw_Terminal_01x02 J3
+L Connector:Screw_Terminal_01x02 J3
 U 1 1 5AC3CE1A
 P 6300 3250
@@
 $EndComp
 $Comp
-L conn:Screw_Terminal_01x02 J4
+L Connector:Screw_Terminal_01x02 J4
 U 1 1 5AC3CE7D
 P 6300 3600
@@
 $EndComp
 $Comp
-L conn:Screw_Terminal_01x02 J5
+L Connector:Screw_Terminal_01x02 J5
 U 1 1 5AC3CED5
 P 6300 3950
@@
 $EndComp
 $Comp
-L device:D D1
+L Device:D D1
 U 1 1 5AB41BB2
 P 2600 3800
@@
 $EndComp
 $Comp
-L conn:Conn_01x04 J1
+L Connector_Generic:Conn_01x04 J1
 U 1 1 5AB40A05
 P 2400 3550
@@
 $EndComp
 $Comp
-L device:Jumper_NC_Dual JP1
+L Device:Jumper_NC_Dual JP1
 U 1 1 5AC3E184
 P 4550 2500
@@
 $EndComp
 $Comp
-L device:Jumper_NC_Dual JP2
+L Device:Jumper_NC_Dual JP2
 U 1 1 5AC3E245
 P 5350 2500
@@
 RX
 $Comp
-L device:R R5
+L Device:R R5
 U 1 1 5AC3F1E0
 P 5200 4950
@@
 $EndComp
 $Comp
-L device:R R4
+L Device:R R4
 U 1 1 5AC3F27A
 P 4950 5050
@@
 	1    0    0    -1
 $EndComp
-Wire Wire Line
-	4950 5200 5300 5200
-Wire Wire Line
-	5300 5100 5200 5100
-Wire Wire Line
-	4800 5100 5200 5100
-Connection ~ 5200 5100
-Wire Wire Line
-	4950 5200 4800 5200
-Connection ~ 4950 5200
 Text GLabel 4800 5100 0    50   Input ~ 0
 TX
 $Comp
-L device:CP C5
+L Device:CP C5
 U 1 1 5AC41046
 P 4550 3600
@@
 $EndComp
 $Comp
-L device:CP C6
+L Device:CP C6
 U 1 1 5AC410CC
 P 5800 3600
@@
 $EndComp
 $Comp
-L conn:Conn_01x03 UART1
+L Connector_Generic:Conn_01x03 UART1
 U 1 1 5AC53A74
 P 3350 4600
@@
 TX
 $Comp
-L conn:Conn_01x04 J6
+L Connector_Generic:Conn_01x04 J6
 U 1 1 5AC544EE
 P 6300 4600
@@
 	1    0    0    -1
 $EndComp
-Wire Wire Line
-	4100 3450 3900 3450
-Connection ~ 3600 3450
-Wire Wire Line
-	3600 3550 3750 3550
-Connection ~ 3600 3550
-$Comp
-L device:R_Small R6
+$Comp
+L Device:R_Small R6
 U 1 1 5AD35758
 P 3750 3350
@@
 	1    0    0    -1
 $EndComp
-Connection ~ 3750 3450
-Wire Wire Line
-	3750 3450 3600 3450
-$Comp
-L device:R_Small R7
+$Comp
+L Device:R_Small R7
 U 1 1 5AD357E7
 P 3750 3650
@@
 	1    0    0    -1
 $EndComp
-Connection ~ 3750 3550
-Wire Wire Line
-	3750 3550 3900 3550
-$Comp
-L device:C_Small C8
+$Comp
+L Device:C_Small C8
 U 1 1 5AD35928
 P 3900 3650
@@
 	1    0    0    -1
 $EndComp
-Connection ~ 3900 3550
-Wire Wire Line
-	3900 3550 4100 3550
-$Comp
-L device:C_Small C7
+$Comp
+L Device:C_Small C7
 U 1 1 5AD359AD
 P 3900 3350
@@
 	1    0    0    -1
 $EndComp
-Connection ~ 3900 3450
-Wire Wire Line
-	3900 3450 3750 3450
 $Comp
 L power:GND #PWR0127
@@
 Text GLabel 4800 5200 0    50   Input ~ 0
 RX
-Wire Wire Line
-	4850 3450 4750 3450
-Connection ~ 4750 3450
-$Comp
-L regul_eigen:L7805SOT89 U1
+$Comp
+L Regulator_Linear:L7805 U1
 U 1 1 5AE0F904
 P 5150 3450
@@
 Wire Wire Line
 	3450 3500 3450 3450
-Connection ~ 3450 3450
 Wire Wire Line
 	3450 3500 3100 3500
@@
 	3100 3500 3100 3550
 Wire Wire Line
-	3450 3550 3200 3550
-Wire Wire Line
 	3200 3550 3200 3450
 Wire Wire Line
 	3200 3450 3100 3450
-Connection ~ 3450 3550
+Wire Wire Line
+	4700 3450 4850 3450
+Wire Wire Line
+	5450 3450 5600 3450
+Wire Wire Line
+	4800 5200 5300 5200
+Wire Wire Line
+	4800 5100 5300 5100
+Wire Wire Line
+	3450 3450 4100 3450
+Wire Wire Line
+	3200 3550 4100 3550
 $EndSCHEMATC
