File: nunchuk_breakout/nunchuk_breakout.kicad_pcb (KiCad board)
At the start: 2 copper layers, 39 x 18 mm, 14 parts, among them J2 Conn_01x04, P1 CONN_WII, U1 L7805SOT89

Commit message: added image
Parts:
- removed the G*** at (107.0, 100.0)
- added G***: LOGO, otter:otterimage_crop_13, B.Cu at (109.4, 99.2)

Commit message: updated PCB
Other:
- board text added: "https://github.com/ Jan--Henrik/hoverboard-breakout"
Changed lines of the file:
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@@
   (general
     (thickness 1.6)
-    (drawings 14)
+    (drawings 15)
     (tracks 27)
     (zones 0)
@@
       (xy -0.203663 2.662024) (xy -0.023791 2.722104) (xy 0.159048 2.738148) (xy 0.3048 2.716815)) (layer B.SilkS) (width 0.01))
   )
+  (gr_text "https://github.com/\nJan--Henrik/hoverboard-breakout" (at 97.2 107.5) (layer F.SilkS)
+    (effects (font (size 0.65 0.62) (thickness 0.11)) (justify left))
+  )
   (gr_text "Hoverboard\nto Nunchuk\nadapter" (at 114 100) (layer F.SilkS)

Commit message: changed rendering
Parts:
- removed C7, C8: 10p, Capacitor_SMD:C_0603_1608Metric
- removed D3: LED, LED_SMD:LED_0805_2012Metric
- removed J2: Conn_01x04, Connector_JST:JST_XH_B04B-XH-A_1x04_P2.50mm_Vertical
- removed R4, R5: 3k3, Resistor_SMD:R_0603_1608Metric
- added C1: 10p, Capacitor_SMD:C_0603_1608Metric, F.Cu at (121.5, 96.5)
- added C2: 10p, Capacitor_SMD:C_0603_1608Metric, F.Cu at (121.5, 103.5)
- added D1: LED, LED_SMD:LED_0805_2012Metric, F.Cu at (105.5, 103.5)
- added J1: Conn_01x04, Connector_JST:JST_XH_B04B-XH-A_1x04_P2.50mm_Vertical, F.Cu at (100.0, 96.2)
- added R1: 220Ohm, Resistor_SMD:R_0603_1608Metric, F.Cu at (109.0, 102.0)
- added R2: 3k3, Resistor_SMD:R_0603_1608Metric, F.Cu at (120.0, 98.0)
- R3: value 220Ohm -> 3k3
- U1: value L7805SOT89 -> L78L33_SOT89; footprint Package_TO_SOT_SMD:SOT-89-3_Handsoldering -> Package_TO_SOT_SMD:SOT-89-3
- moved R3 11.0 mm to (120.0, 101.8), turned to 270 degrees
- moved C3 6.00 mm to (105.0, 94.5)
- moved C4 6.00 mm to (108.0, 94.5)
- moved U1 2.28 mm to (106.5, 98.3), turned to 270 degrees
- moved G*** 0.46 mm to (109.5, 98.8)
Connections:
- R3 pad 1: Net-(D3-Pad2) -> VCC
- R3 pad 2: VCC -> SCL
- U1 pad 1: VDD -> VCC
- U1 pad 3: VCC -> VDD
Routing:
- net Net-(D1-Pad2): track 0.00 -> 3.07 mm
- net Net-(D3-Pad2): track 2.19 -> 0.00 mm
- net GND: vias 5 -> 4
