File: nunchuk_breakout/nunchuk_breakout.sch (KiCad schematic (older format))
At the start: 13 parts, among them J2 Conn_01x04, P1 CONN_WII, U1 L7805SOT89

Commit message: changed rendering
Parts:
- removed U1: L7805SOT89, Package_TO_SOT_SMD:SOT-89-3_Handsoldering, symbol Regulator_Linear:L7805
- added U1: L78L33_SOT89, Package_TO_SOT_SMD:SOT-89-3, symbol Regulator_Linear:L78L33_SOT89
- renumbered C8 to C1, C7 to C2, D3 to D1, J2 to J1, R3 to R1, R4 to R2, R5 to R3
Changed lines of the file:
@@
 $EndComp
 $Comp
-L Connector_Generic:Conn_01x04 J2
+L Connector_Generic:Conn_01x04 J1
 U 1 1 5AB40975
 P 2150 3550
-F 0 "J2" H 2070 3125 50  0000 C CNN
+F 0 "J1" H 2070 3125 50  0000 C CNN
 F 1 "Conn_01x04" H 2070 3216 50  0000 C CNN
 F 2 "Connector_JST:JST_XH_B04B-XH-A_1x04_P2.50mm_Vertical" H 2150 3550 50  0001 C CNN
@@
 $EndComp
 $Comp
-L power:GND #PWR0102
+L power:GND #PWR03
 U 1 1 5AB40AE8
 P 2350 3350
-F 0 "#PWR0102" H 2350 3100 50  0001 C CNN
+F 0 "#PWR03" H 2350 3100 50  0001 C CNN
 F 1 "GND" H 2355 3177 50  0000 C CNN
 F 2 "" H 2350 3350 50  0001 C CNN
@@
 $EndComp
 $Comp
-L power:GND #PWR0103
+L power:GND #PWR012
 U 1 1 5AB40B19
 P 4050 3650
-F 0 "#PWR0103" H 4050 3400 50  0001 C CNN
+F 0 "#PWR012" H 4050 3400 50  0001 C CNN
 F 1 "GND" H 4055 3477 50  0000 C CNN
 F 2 "" H 4050 3650 50  0001 C CNN
@@
 $EndComp
 $Comp
-L power:GND #PWR0104
+L power:GND #PWR013
 U 1 1 5AB40B4A
 P 4550 3650
-F 0 "#PWR0104" H 4550 3400 50  0001 C CNN
+F 0 "#PWR013" H 4550 3400 50  0001 C CNN
 F 1 "GND" H 4555 3477 50  0000 C CNN
 F 2 "" H 4550 3650 50  0001 C CNN
@@
 $EndComp
 $Comp
-L power:GND #PWR0105
+L power:GND #PWR014
 U 1 1 5AB40B94
 P 5000 3650
-F 0 "#PWR0105" H 5000 3400 50  0001 C CNN
+F 0 "#PWR014" H 5000 3400 50  0001 C CNN
 F 1 "GND" H 5005 3477 50  0000 C CNN
 F 2 "" H 5000 3650 50  0001 C CNN
@@
 $EndComp
 $Comp
-L power:VCC #PWR0106
+L power:VCC #PWR015
 U 1 1 5AB40C12
 P 5100 3350
-F 0 "#PWR0106" H 5100 3200 50  0001 C CNN
+F 0 "#PWR015" H 5100 3200 50  0001 C CNN
 F 1 "VCC" H 5117 3523 50  0000 C CNN
 F 2 "" H 5100 3350 50  0001 C CNN
@@
 $EndComp
 $Comp
-L power:VDD #PWR0107
+L power:VDD #PWR011
 U 1 1 5AB40CD6
 P 3950 3350
-F 0 "#PWR0107" H 3950 3200 50  0001 C CNN
+F 0 "#PWR011" H 3950 3200 50  0001 C CNN
 F 1 "VDD" H 3967 3523 50  0000 C CNN
 F 2 "" H 3950 3350 50  0001 C CNN
@@
 $EndComp
 $Comp
-L power:VDD #PWR0108
+L power:VDD #PWR04
 U 1 1 5AB40D07
 P 2350 3650
-F 0 "#PWR0108" H 2350 3500 50  0001 C CNN
+F 0 "#PWR04" H 2350 3500 50  0001 C CNN
 F 1 "VDD" H 2367 3823 50  0000 C CNN
 F 2 "" H 2350 3650 50  0001 C CNN
@@
 SDA
 $Comp
-L Device:LED D3
+L Device:LED D1
 U 1 1 5AB41F7D
 P 1400 3750
-F 0 "D3" H 1392 3495 50  0000 C CNN
+F 0 "D1" H 1392 3495 50  0000 C CNN
 F 1 "LED" H 1392 3586 50  0000 C CNN
 F 2 "LED_SMD:LED_0805_2012Metric" H 1400 3750 50  0001 C CNN
@@
 $EndComp
 $Comp
-L Device:R R3
+L Device:R R1
 U 1 1 5AB42057
 P 1400 3400
-F 0 "R3" V 1193 3400 50  0000 C CNN
+F 0 "R1" V 1193 3400 50  0000 C CNN
 F 1 "220Ohm" V 1284 3400 50  0000 C CNN
 F 2 "Resistor_SMD:R_0603_1608Metric" V 1330 3400 50  0001 C CNN
@@
 $EndComp
 $Comp
-L power:GND #PWR0116
+L power:GND #PWR02
 U 1 1 5AB420F1
 P 1400 3900
-F 0 "#PWR0116" H 1400 3650 50  0001 C CNN
+F 0 "#PWR02" H 1400 3650 50  0001 C CNN
 F 1 "GND" H 1405 3727 50  0000 C CNN
 F 2 "" H 1400 3900 50  0001 C CNN
@@
 $EndComp
 $Comp
-L power:VCC #PWR0117
+L power:VCC #PWR01
 U 1 1 5AB42144
 P 1400 3250
-F 0 "#PWR0117" H 1400 3100 50  0001 C CNN
+F 0 "#PWR01" H 1400 3100 50  0001 C CNN
 F 1 "VCC" H 1417 3423 50  0000 C CNN
 F 2 "" H 1400 3250 50  0001 C CNN
@@
 SCL
 $Comp
-L Device:R R5
+L Device:R R3
 U 1 1 5AC3F1E0
 P 3200 4550
-F 0 "R5" H 3270 4596 50  0000 L CNN
+F 0 "R3" H 3270 4596 50  0000 L CNN
 F 1 "3k3" H 3270 4505 50  0000 L CNN
 F 2 "Resistor_SMD:R_0603_1608Metric" V 3130 4550 50  0001 C CNN
@@
 $EndComp
 $Comp
-L Device:R R4
+L Device:R R2
 U 1 1 5AC3F27A
 P 2850 4550
-F 0 "R4" H 2920 4596 50  0000 L CNN
+F 0 "R2" H 2920 4596 50  0000 L CNN
 F 1 "3k3" H 2920 4505 50  0000 L CNN
 F 2 "Resistor_SMD:R_0603_1608Metric" V 2780 4550 50  0001 C CNN
@@
 $EndComp
 $Comp
-L power:VCC #PWR0122
+L power:VCC #PWR07
 U 1 1 5AC3F35A
 P 2850 4400
-F 0 "#PWR0122" H 2850 4250 50  0001 C CNN
+F 0 "#PWR07" H 2850 4250 50  0001 C CNN
 F 1 "VCC" H 2867 4573 50  0000 C CNN
 F 2 "" H 2850 4400 50  0001 C CNN
@@
 $EndComp
 $Comp
-L power:VCC #PWR0123
+L power:VCC #PWR08
 U 1 1 5AC3F3BB
 P 3200 4400
-F 0 "#PWR0123" H 3200 4250 50  0001 C CNN
+F 0 "#PWR08" H 3200 4250 50  0001 C CNN
 F 1 "VCC" H 3217 4573 50  0000 C CNN
 F 2 "" H 3200 4400 50  0001 C CNN
@@
 $EndComp
 $Comp
-L Device:C_Small C8
+L Device:C_Small C1
 U 1 1 5AD35928
 P 2850 3300
-F 0 "C8" H 2942 3346 50  0000 L CNN
+F 0 "C1" H 2942 3346 50  0000 L CNN
 F 1 "10p" H 2942 3255 50  0000 L CNN
 F 2 "Capacitor_SMD:C_0603_1608Metric" H 2850 3300 50  0001 C CNN
@@
 $EndComp
 $Comp
-L Device:C_Small C7
+L Device:C_Small C2
 U 1 1 5AD359AD
 P 2850 3700
-F 0 "C7" H 2942 3746 50  0000 L CNN
+F 0 "C2" H 2942 3746 50  0000 L CNN
 F 1 "10p" H 2942 3655 50  0000 L CNN
 F 2 "Capacitor_SMD:C_0603_1608Metric" H 2850 3700 50  0001 C CNN
@@
 $EndComp
 $Comp
-L power:GND #PWR0127
+L power:GND #PWR06
 U 1 1 5AD35A84
 P 2850 3800
-F 0 "#PWR0127" H 2850 3550 50  0001 C CNN
+F 0 "#PWR06" H 2850 3550 50  0001 C CNN
 F 1 "GND" H 2855 3627 50  0000 C CNN
 F 2 "" H 2850 3800 50  0001 C CNN
@@
 $EndComp
 $Comp
-L power:GND #PWR0130
+L power:GND #PWR05
 U 1 1 5AD35C56
 P 2850 3200
-F 0 "#PWR0130" H 2850 2950 50  0001 C CNN
+F 0 "#PWR05" H 2850 2950 50  0001 C CNN
 F 1 "GND" H 2855 3027 50  0000 C CNN
 F 2 "" H 2850 3200 50  0001 C CNN
@@
 Text GLabel 2850 4700 3    50   Input ~ 0
 SDA
-$Comp
-L Regulator_Linear:L7805 U1
-U 1 1 5AE0F904
-P 4550 3350
-F 0 "U1" H 4550 3592 50  0000 C CNN
-F 1 "L7805SOT89" H 4550 3501 50  0000 C CNN
-F 2 "Package_TO_SOT_SMD:SOT-89-3_Handsoldering" H 4575 3200 50  0001 L CIN
-F 3 "http://www.st.com/content/ccc/resource/technical/document/datasheet/41/4f/b3/b0/12/d4/47/88/CD00000444.pdf/files/CD00000444.pdf/jcr:content/translations/en.CD00000444.pdf" H 4550 3300 50  0001 C CNN
-	1    4550 3350
-	1    0    0    -1
-$EndComp
 Wire Wire Line
 	2350 3450 2850 3450
@@
 $EndComp
 $Comp
-L power:VCC #PWR0109
+L power:VCC #PWR09
 U 1 1 5C2CB62A
 P 3350 1900
-F 0 "#PWR0109" H 3350 1750 50  0001 C CNN
+F 0 "#PWR09" H 3350 1750 50  0001 C CNN
 F 1 "VCC" H 3367 2073 50  0000 C CNN
 F 2 "" H 3350 1900 50  0001 C CNN
@@
 $EndComp
 $Comp
-L power:GND #PWR0111
+L power:GND #PWR010
 U 1 1 5C2CB79A
 P 3350 2100
-F 0 "#PWR0111" H 3350 1850 50  0001 C CNN
+F 0 "#PWR010" H 3350 1850 50  0001 C CNN
 F 1 "GND" H 3355 1927 50  0000 C CNN
 F 2 "" H 3350 2100 50  0001 C CNN
@@
 Wire Wire Line
 	2850 3450 3350 3450
+$Comp
+L Regulator_Linear:L78L33_SOT89 U1
+U 1 1 5C2CD9F6
+P 4550 3350
+F 0 "U1" H 4550 3592 50  0000 C CNN
+F 1 "L78L33_SOT89" H 4550 3501 50  0000 C CNN
+F 2 "Package_TO_SOT_SMD:SOT-89-3" H 4550 3550 50  0001 C CIN
+F 3 "http://www.st.com/content/ccc/resource/technical/document/datasheet/15/55/e5/aa/23/5b/43/fd/CD00000446.pdf/files/CD00000446.pdf/jcr:content/translations/en.CD00000446.pdf" H 4550 3300 50  0001 C CNN
+	1    4550 3350
+	1    0    0    -1
+$EndComp
 $EndSCHEMATC
